Commit message: Fixed rviz launch

File: tractor_sim_description/urdf/kubo_macros.urdf.xacro (robot description, xacro)
@@ -1,18 +1,18 @@
 <?xml version="1.0"?>
-<robot>
+<robot xmlns:xacro="http://www.ros.org/wiki/xacro">
   <!-- Null inertial element. This is needed to make the model work with
        Gazebo. -->
-  <macro name="null_inertial">
+  <xacro:macro name="null_inertial">
     <inertial>
       <mass value="0.001"/>
       <inertia ixx="0.001" ixy="0" ixz="0" iyy="0.001" iyz="0" izz="0.001"/>
     </inertial>
-  </macro>
+  </xacro:macro>
   <!-- Inertia of a solid cuboid. Width is measured along the x axis, depth
        along the y axis, and height along the z axis. -->
-  <macro name="solid_cuboid_inertial"
+  <xacro:macro name="solid_cuboid_inertial"
                params="width depth height mass *origin">
     <inertial>
-      <insert_block name="origin"/>
+      <xacro:insert_block name="origin"/>
       <mass value="${mass}"/>
       <inertia ixx="${mass * (depth * depth + height * height) / 12}"
@@ -22,9 +22,9 @@
                izz="${mass * (width * width + depth * depth) / 12}"/>
     </inertial>
-  </macro>
+  </xacro:macro>
   <!-- Inertia of a thick-walled cylindrical tube with open ends. Height is
        measured along the z axis, which is the tube's axis. inner_rad and
        outer_rad are the tube's inner and outer radii, respectively. -->
-  <macro name="thick_walled_tube_inertial"
+  <xacro:macro name="thick_walled_tube_inertial"
                params="inner_rad outer_rad height mass">
     <inertial>
@@ -39,7 +39,7 @@
                     outer_rad * outer_rad) / 2}"/>
     </inertial>
-  </macro>
+  </xacro:macro>
   <!-- Shock absorber -->
-  <macro name="bshock"
+  <xacro:macro name="bshock"
                params="lr_prefix fr_prefix lr_reflect fr_reflect child">
     <joint name="${lr_prefix}_${fr_prefix}_shock" type="prismatic">
@@ -67,6 +67,6 @@
       </actuator>
     </transmission>
-  </macro>
-  <macro name="fshock"
+  </xacro:macro>
+  <xacro:macro name="fshock"
                params="lr_prefix fr_prefix lr_reflect fr_reflect child">
     <joint name="${lr_prefix}_${fr_prefix}_shock" type="prismatic">
@@ -94,7 +94,7 @@
       </actuator>
     </transmission>
-  </macro>
+  </xacro:macro>
   <!-- The "wheel" macro defines an axle carrier, axle, and wheel. -->
-  <macro name="wheel" params="lr_prefix fr_prefix lr_reflect tire_dia tire_width hex_hub_depth wheel_mass">
+  <xacro:macro name="wheel" params="lr_prefix fr_prefix lr_reflect tire_dia tire_width hex_hub_depth wheel_mass">
     <link name="${lr_prefix}_${fr_prefix}_axle_carrier">
       <null_inertial/>
@@ -148,7 +148,7 @@
       <material>Gazebo/Black</material>
     </gazebo>
-  </macro>
+  </xacro:macro>
   <!-- Front wheel -->
-  <macro name="front_wheel"
+  <xacro:macro name="front_wheel"
                params="lr_prefix fr_prefix lr_reflect fr_reflect">
     <fshock lr_prefix="${lr_prefix}" fr_prefix="${fr_prefix}"
@@ -181,7 +181,7 @@
                  tire_dia="${ftire_dia}" tire_width="${ftire_width}"
                  hex_hub_depth="${fhex_hub_depth}" wheel_mass="${fwheel_mass}"/>
-  </macro>
+  </xacro:macro>
   <!-- Rear wheel -->
-  <macro name="rear_wheel"
+  <xacro:macro name="rear_wheel"
                params="lr_prefix fr_prefix lr_reflect fr_reflect">
     <bshock lr_prefix="${lr_prefix}" fr_prefix="${fr_prefix}"
@@ -192,6 +192,6 @@
                  tire_dia="${btire_dia}" tire_width="${btire_width}"
                  hex_hub_depth="${bhex_hub_depth}" wheel_mass="${bwheel_mass}"/>
-  </macro>
-  <macro name="sensor"
+  </xacro:macro>
+  <xacro:macro name="sensor"
          params = "sensor_name x_pos y_pos z_pos x_rot y_rot z_rot">
      <link name="${sensor_name}">
@@ -222,4 +222,4 @@
        <child link="${sensor_name}"/>
      </joint>
-  </macro>
+  </xacro:macro>
 </robot>

File: tractor_sim_description/urdf/kubo_materials.urdf.xacro (robot description, xacro)
@@ -1,4 +1,4 @@
 <?xml version="1.0"?>
-<robot>
+<robot xmlns:xacro="http://www.ros.org/wiki/xacro">
   <material name="chassis_mat">
     <color rgba="0.5 0.5 0.5 1"/>
