Commit message: Dimensions ~90% accurate, front wheels still need modification

File: tractor_sim_description/urdf/kubo.urdf.xacro (robot description, xacro)
@@ -6,20 +6,8 @@
   <!-- chassis_length is measured along the x axis, chassis_width
        along the y axis, and chassis_height along the z axis. -->
-  <xacro:property name="chassis_length" value="0.258"/>
-  <xacro:property name="chassis_width" value="0.168"/>
-  <xacro:property name="chassis_height" value="0.01"/>
+  <xacro:property name="chassis_length" value="1.5"/>
+  <xacro:property name="chassis_width" value="0.6"/>
+  <xacro:property name="chassis_height" value="0.1"/>
   <xacro:property name="chassis_mass" value="2.788"/>
-  <!-- battery_dist is the distance between the inner edges of the
-       batteries. battery_comp_depth is the battery compartment depth.
-       battery_length is measured along the x axis, battery_width
-       along the y axis, and battery_height along the z axis. -->
-  <xacro:property name="battery_x_offset" value="0.055"/>
-  <xacro:property name="battery_dist" value="0.065"/>
-  <xacro:property name="battery_comp_depth" value="0.02"/>
-  <xacro:property name="battery_comp_angle" value="0.34906585"/>
-  <xacro:property name="battery_length" value="0.16"/>
-  <xacro:property name="battery_width" value="0.047"/>
-  <xacro:property name="battery_height" value="0.024"/>
-  <xacro:property name="battery_mass" value="0.5025"/>
   <!-- hub_dia and tire_dia are the diameters of the hub and tire,
        respectively. hex_hub_depth is the distance that the hex hub is
@@ -28,7 +16,7 @@
        axle_length. -->
   <xacro:property name="hub_dia" value="0.09652"/>
-  <xacro:property name="tire_dia" value="0.14605"/>
-  <xacro:property name="tire_width" value="0.0889"/>
-  <xacro:property name="hex_hub_depth" value="0.01445"/>
+  <xacro:property name="tire_dia" value="0.7"/>
+  <xacro:property name="tire_width" value="0.2"/>
+  <xacro:property name="hex_hub_depth" value="${tire_width / 2 - axle_length}"/> <!-- tire_width / 2 - axle_length-->
   <xacro:property name="wheel_mass" value="0.29"/>
   <!-- hex_hub_dist is the distance between left and right hex hubs when
@@ -36,7 +24,7 @@
        from a U joint to the corresponding hex hub. wheel_travel is the
        vertical wheel travel. -->
-  <xacro:property name="wheelbase" value="0.335"/>
-  <xacro:property name="hex_hub_dist" value="0.365"/>
-  <xacro:property name="axle_length" value="0.03"/>
+  <xacro:property name="wheelbase" value="1.5"/>
+  <xacro:property name="hex_hub_dist" value="1.4"/>
+  <xacro:property name="axle_length" value="0.3"/>
   <xacro:property name="wheel_travel" value="0.084"/>
   <xacro:property name="shock_z_offset" value="0.0655"/>
@@ -45,6 +33,6 @@
        of a Traxxas Ultra Shock shock absorber spring's constant, is
        437.817 N/m. -->
-  <xacro:property name="shock_eff_limit" value="12.5106"/>
-  <xacro:property name="shock_vel_limit" value="1000"/>
+  <xacro:property name="shock_eff_limit" value="125106"/>
+  <xacro:property name="shock_vel_limit" value="1000000"/>
   <!-- The specifications for a Titan(R) 550 motor could not be found, so the
        stall torque of a Mabuchi Motor(R) RS-550VC-7525 motor was used instead.
@@ -59,14 +47,11 @@
        axle_vel_limit = (2 * pi) * (max_speed / (pi * tire_dia)) =
          244.8696 rad/s -->
-  <xacro:property name="axle_eff_limit" value="5.12766"/>
-  <xacro:property name="axle_vel_limit" value="244.8696"/>
+  <xacro:property name="axle_eff_limit" value="512766"/>
+  <xacro:property name="axle_vel_limit" value="2448696"/>
   <!-- These constants are used to simulate a Traxxas 2056 servo operated at
        6 V. servo_stall_torque is measured in N m. servo_no_load_speed is
        measured in rad/s. -->
-  <xacro:property name="servo_stall_torque" value="0.5649"/>
-  <xacro:property name="servo_no_load_speed" value="4.553"/>
-  <material name="battery_mat">
-    <color rgba="0 0 1 1"/>
-  </material>
+  <xacro:property name="servo_stall_torque" value="5649"/>
+  <xacro:property name="servo_no_load_speed" value="4553"/>
   <material name="chassis_mat">
     <color rgba="0.5 0.5 0.5 1"/>
@@ -113,46 +98,4 @@
                     outer_rad * outer_rad) / 2}"/>
     </inertial>
-  </xacro:macro>
-  <!-- Battery -->
-  <xacro:macro name="battery" params="prefix reflect">
-    <joint name="chassis_to_${prefix}_battery" type="fixed">
-      <parent link="chassis"/>
-      <child link="${prefix}_battery_offset"/>
-      <origin xyz="${battery_x_offset - battery_length / 2}
-                   ${reflect * battery_dist / 2}
-                   0"
-              rpy="${reflect * battery_comp_angle} 0 0"/>
-    </joint>
-    <link name="${prefix}_battery_offset">
-      <xacro:null_inertial/>
-    </link>
-    <joint name="offset_to_${prefix}_battery" type="fixed">
-      <parent link="${prefix}_battery_offset"/>
-      <child link="${prefix}_battery"/>
-      <origin xyz="0
-                   ${reflect * battery_width / 2}
-                   ${(battery_height / 2) - battery_comp_depth}"/>
-    </joint>
-    <link name="${prefix}_battery">
-      <visual>
-        <geometry>
-          <box size="${battery_length} ${battery_width} ${battery_height}"/>
-        </geometry>
-        <material name="battery_mat"/>
-      </visual>
-      <collision>
-        <geometry>
-          <box size="${battery_length} ${battery_width} ${battery_height}"/>
-        </geometry>
-      </collision>
-      <xacro:solid_cuboid_inertial
-         width="${battery_length}" depth="${battery_width}"
-         height="${battery_height}" mass="${battery_mass}">
-        <origin/>
-      </xacro:solid_cuboid_inertial>
-    </link>
-    <gazebo reference="${prefix}_battery">
-      <material>Gazebo/Blue</material>
-    </gazebo>
   </xacro:macro>
   <!-- Shock absorber -->
@@ -317,7 +260,4 @@
     <child link="chassis"/>
   </joint>
-  <!-- Batteries -->
-  <xacro:battery prefix="left" reflect="1"/>
-  <xacro:battery prefix="right" reflect="-1"/>
   <!-- Wheels -->
   <xacro:front_wheel lr_prefix="left" fr_prefix="front"

Commit message: Made small front wheels

File: tractor_sim_description/urdf/kubo.urdf.xacro (robot description, xacro)
@@ -15,9 +15,13 @@
        is a "zero offset" wheel. hex_hub_depth = tire_width / 2 -
        axle_length. -->
-  <xacro:property name="hub_dia" value="0.09652"/>
-  <xacro:property name="tire_dia" value="0.7"/>
-  <xacro:property name="tire_width" value="0.2"/>
-  <xacro:property name="hex_hub_depth" value="${tire_width / 2 - axle_length}"/> <!-- tire_width / 2 - axle_length-->
-  <xacro:property name="wheel_mass" value="0.29"/>
+  <xacro:property name="hub_dia" value="0.09652"/> <!-- ? -->
+  <xacro:property name="ftire_dia" value="0.5"/>
+  <xacro:property name="ftire_width" value="0.15"/>
+  <xacro:property name="fhex_hub_depth" value="${ftire_width / 2 - axle_length}"/> <!-- tire_width / 2 - axle_length-->
+  <xacro:property name="fwheel_mass" value="0.29"/>
+  <xacro:property name="btire_dia" value="0.7"/>
+  <xacro:property name="btire_width" value="0.2"/>
+  <xacro:property name="bhex_hub_depth" value="${btire_width / 2 - axle_length}"/> <!-- tire_width / 2 - axle_length-->
+  <xacro:property name="bwheel_mass" value="0.29"/>
   <!-- hex_hub_dist is the distance between left and right hex hubs when
        the shock absorbers are fully extended. axle_length is the distance
@@ -25,7 +29,7 @@
        vertical wheel travel. -->
   <xacro:property name="wheelbase" value="1.5"/>
-  <xacro:property name="hex_hub_dist" value="1.4"/>
-  <xacro:property name="axle_length" value="0.3"/>
-  <xacro:property name="wheel_travel" value="0.084"/>
+  <xacro:property name="hex_hub_dist" value="1.4"/> <!-- ? -->
+  <xacro:property name="axle_length" value="0.3"/> <!-- ? -->
+  <xacro:property name="wheel_travel" value="0"/>
   <xacro:property name="shock_z_offset" value="0.0655"/>
   <!-- shock_eff_limit is 2 * ((shock_stroke / 2) * shock_spring_constant) N.
@@ -126,5 +130,5 @@
   </xacro:macro>
   <!-- The "wheel" macro defines an axle carrier, axle, and wheel. -->
-  <xacro:macro name="wheel" params="lr_prefix fr_prefix lr_reflect">
+  <xacro:macro name="wheel" params="lr_prefix fr_prefix lr_reflect tire_dia tire_width hex_hub_depth wheel_mass">
     <link name="${lr_prefix}_${fr_prefix}_axle_carrier">
       <xacro:null_inertial/>
@@ -208,5 +212,7 @@
     </transmission>
     <xacro:wheel lr_prefix="${lr_prefix}" fr_prefix="${fr_prefix}"
-                 lr_reflect="${lr_reflect}"/>
+                 lr_reflect="${lr_reflect}"
+                 tire_dia="${ftire_dia}" tire_width="${ftire_width}"
+                 hex_hub_depth="${fhex_hub_depth}" wheel_mass="${fwheel_mass}"/>
   </xacro:macro>
   <!-- Rear wheel -->
@@ -217,5 +223,7 @@
                  child="${lr_prefix}_${fr_prefix}_axle_carrier"/>
     <xacro:wheel lr_prefix="${lr_prefix}" fr_prefix="${fr_prefix}"
-                 lr_reflect="${lr_reflect}"/>
+                 lr_reflect="${lr_reflect}"
+                 tire_dia="${btire_dia}" tire_width="${btire_width}"
+                 hex_hub_depth="${bhex_hub_depth}" wheel_mass="${bwheel_mass}"/>
   </xacro:macro>
   <!-- base_link must have geometry so that its axes can be displayed in

Commit message: Adding correctly dimensioned sim

File: tractor_sim_description/urdf/kubo.urdf.xacro (robot description, xacro)
@@ -1,4 +1,5 @@
 <?xml version="1.0"?>
 <robot name="kubo" xmlns:xacro="http://www.ros.org/wiki/xacro">
+  <xacro:include filename="$(find hector_sensors_description)/urdf/hokuyo_utm30lx.urdf.xacro"/>
   <!-- Degree-to-radian conversions -->
   <xacro:property name="degrees_45" value="0.785398163"/>
@@ -119,10 +120,10 @@
       <type>transmission_interface/SimpleTransmission</type>
       <joint name="${lr_prefix}_${fr_prefix}_shock">
-        <hardwareInterface>EffortJointInterface</hardwareInterface>
+        <hardwareInterface>hardware_interface/EffortJointInterface</hardwareInterface>
       </joint>
       <actuator name="${lr_prefix}_${fr_prefix}_shock_act">
         <!-- This hardwareInterface element exists for compatibility
              with ROS Hydro. -->
-        <hardwareInterface>EffortJointInterface</hardwareInterface>
+        <hardwareInterface>hardware_interface/EffortJointInterface</hardwareInterface>
         <mechanicalReduction>1</mechanicalReduction>
       </actuator>
@@ -146,10 +147,10 @@
       <type>transmission_interface/SimpleTransmission</type>
       <joint name="${lr_prefix}_${fr_prefix}_axle">
-        <hardwareInterface>EffortJointInterface</hardwareInterface>
+        <hardwareInterface>hardware_interface/EffortJointInterface</hardwareInterface>
       </joint>
       <actuator name="${lr_prefix}_${fr_prefix}_axle_act">
         <!-- This hardwareInterface element exists for compatibility
              with ROS Hydro. -->
-        <hardwareInterface>EffortJointInterface</hardwareInterface>
+        <hardwareInterface>hardware_interface/EffortJointInterface</hardwareInterface>
         <mechanicalReduction>1</mechanicalReduction>
       </actuator>
@@ -202,10 +203,10 @@
       <type>transmission_interface/SimpleTransmission</type>
       <joint name="${lr_prefix}_steering_joint">
-        <hardwareInterface>EffortJointInterface</hardwareInterface>
+        <hardwareInterface>hardware_interface/EffortJointInterface</hardwareInterface>
       </joint>
       <actuator name="${lr_prefix}_steering_act">
         <!-- This hardwareInterface element exists for compatibility
              with ROS Hydro. -->
-        <hardwareInterface>EffortJointInterface</hardwareInterface>
+        <hardwareInterface>hardware_interface/EffortJointInterface</hardwareInterface>
         <mechanicalReduction>1</mechanicalReduction>
       </actuator>
@@ -245,7 +246,6 @@
       <origin xyz="0 0 ${-chassis_height / 2}"/>
       <geometry>
-        <box size="${chassis_length} ${chassis_width} ${chassis_height}"/>
+        <mesh scale="1 1 1" filename="package://tractor_sim_description/meshes/Chassis.stl"/>
       </geometry>
-      <material name="chassis_mat"/>
     </visual>
     <collision>
@@ -280,3 +280,6 @@
     <plugin name="gazebo_ros_control" filename="libgazebo_ros_control.so"/>
   </gazebo>
+  <hokuyo_utm30lx_model name="hokuyo_laser" parent="base_link">
+    <origin xyz="0 0 +0.30" rpy="0 0 0" />
+  </hokuyo_utm30lx_model>
 </robot>

Commit message: Fixing mesh

File: tractor_sim_description/urdf/kubo.urdf.xacro (robot description, xacro)
@@ -246,6 +246,7 @@
       <origin xyz="0 0 ${-chassis_height / 2}"/>
       <geometry>
-        <mesh scale="1 1 1" filename="package://tractor_sim_description/meshes/Chassis.stl"/>
+        <box size="${chassis_length} ${chassis_width} ${chassis_height}"/>
       </geometry>
+      <material name="chassis_mat"/>
     </visual>
     <collision>

Commit message: Added sensors

File: tractor_sim_description/urdf/kubo.urdf.xacro (robot description, xacro)
@@ -1,5 +1,5 @@
 <?xml version="1.0"?>
 <robot name="kubo" xmlns:xacro="http://www.ros.org/wiki/xacro">
-  <xacro:include filename="$(find hector_sensors_description)/urdf/hokuyo_utm30lx.urdf.xacro"/>
+  <xacro:include filename="$(find tractor_sim_description)/urdf/kubo.gazebo" />
   <!-- Degree-to-radian conversions -->
   <xacro:property name="degrees_45" value="0.785398163"/>
@@ -59,4 +59,6 @@
   <xacro:property name="servo_stall_torque" value="5649"/>
   <xacro:property name="servo_no_load_speed" value="4553"/>
+  <xacro:property name="cameraSize" value="0.05"/>
+  <xacro:property name="cameraMass" value="0.1"/>
   <material name="chassis_mat">
     <color rgba="0.5 0.5 0.5 1"/>
@@ -281,6 +283,56 @@
     <plugin name="gazebo_ros_control" filename="libgazebo_ros_control.so"/>
   </gazebo>
-  <hokuyo_utm30lx_model name="hokuyo_laser" parent="base_link">
-    <origin xyz="0 0 +0.30" rpy="0 0 0" />
-  </hokuyo_utm30lx_model>
+  <link name="camera">
+    <collision>
+      <origin xyz="0 0 0" rpy="0 0 0"/>
+      <geometry>
+        <box size="${cameraSize} ${cameraSize} ${cameraSize}"/>
+      </geometry>
+    </collision>
+    <visual>
+      <origin xyz="0 0 0" rpy="0 0 0"/>
+      <geometry>
+        <box size="${cameraSize} ${cameraSize} ${cameraSize}"/>
+      </geometry>
+      <material name="green"/>
+    </visual>
+    <inertial>
+      <mass value="${cameraMass}" />
+      <origin xyz="0 0 0" rpy="0 0 0"/>
+      <box_inertia m="${cameraMass}" x="${cameraSize}" y="${cameraSize}" z="${cameraSize}" />
+      <inertia ixx="1e-6" ixy="0" ixz="0" iyy="1e-6" iyz="0" izz="1e-6" />
+    </inertial>
+  </link>
+  <joint name="camera_joint" type="fixed">
+    <axis xyz="0 1 0" />
+    <origin xyz=".2 0 .3" rpy="0 0 0"/> <!-- CHANGE LATER-->
+    <parent link="chassis"/>
+    <child link="camera"/>
+  </joint>
+  <joint name="hokuyo_joint" type="fixed">
+    <axis xyz="0 1 0" />
+    <origin xyz=".15 0 .2" rpy="0 -.1 0"/> <!-- CHANGE LATER-->
+    <parent link="chassis"/>
+    <child link="hokuyo"/>
+  </joint>
+  <!-- Hokuyo Laser -->
+  <link name="hokuyo">
+    <collision>
+      <origin xyz="0 0 0" rpy="0 0 0"/>
+      <geometry>
+    <box size="0.1 0.1 0.1"/>
+      </geometry>
+    </collision>
+    <visual>
+      <origin xyz="0 0 0" rpy="0 0 0"/>
+      <geometry>
+        <mesh filename="package://tractor_sim_description/meshes/hokuyo.dae"/>
+      </geometry>
+    </visual>
+    <inertial>
+      <mass value="1e-5" />
+      <origin xyz="0 0 0" rpy="0 0 0"/>
+      <inertia ixx="1e-6" ixy="0" ixz="0" iyy="1e-6" iyz="0" izz="1e-6" />
+    </inertial>
+  </link>
 </robot>
