Commit message: Moved base link, figured out chassis orientation

File: tractor_sim_description/urdf/kubo.urdf.xacro (robot description, xacro)
@@ -1,14 +1,18 @@
 <?xml version="1.0"?>
 <robot name="kubo" xmlns:xacro="http://www.ros.org/wiki/xacro">
-  <xacro:include filename="$(find tractor_sim_description)/urdf/kubo.gazebo" />
+  <xacro:include filename="$(find tractor_sim_description)/urdf/kubo.gazebo"/>
+  <xacro:include filename="$(find tractor_sim_description)/urdf/kubo_materials.urdf.xacro"/>
+  <xacro:include filename="$(find tractor_sim_description)/urdf/kubo_macros.urdf.xacro"/>
   <!-- Degree-to-radian conversions -->
   <xacro:property name="degrees_45" value="0.785398163"/>
   <xacro:property name="degrees_90" value="1.57079633"/>
   <!-- chassis_length is measured along the x axis, chassis_width
-       along the y axis, and chassis_height along the z axis. -->
+       along the y axis, and chassis_height along the z axis.
+      Note: Size of chassis won't affect wheel position or function-->
   <xacro:property name="chassis_length" value="1.5"/>
   <xacro:property name="chassis_width" value="0.6"/>
   <xacro:property name="chassis_height" value="0.1"/>
   <xacro:property name="chassis_mass" value="2.788"/>
+  <xacro:property name="chassis_offset" value=".25"/> <!-- Z Distance from ground -->
   <!-- hub_dia and tire_dia are the diameters of the hub and tire,
        respectively. hex_hub_depth is the distance that the hex hub is
@@ -61,173 +65,4 @@
   <xacro:property name="cameraSize" value="0.05"/>
   <xacro:property name="cameraMass" value="0.1"/>
-  <material name="chassis_mat">
-    <color rgba="0.5 0.5 0.5 1"/>
-  </material>
-  <material name="tire_mat">
-    <color rgba="0 0 0 1"/>
-  </material>
-  <!-- Null inertial element. This is needed to make the model work with
-       Gazebo. -->
-  <xacro:macro name="null_inertial">
-    <inertial>
-      <mass value="0.001"/>
-      <inertia ixx="0.001" ixy="0" ixz="0" iyy="0.001" iyz="0" izz="0.001"/>
-    </inertial>
-  </xacro:macro>
-  <!-- Inertia of a solid cuboid. Width is measured along the x axis, depth
-       along the y axis, and height along the z axis. -->
-  <xacro:macro name="solid_cuboid_inertial"
-               params="width depth height mass *origin">
-    <inertial>
-      <xacro:insert_block name="origin"/>
-      <mass value="${mass}"/>
-      <inertia ixx="${mass * (depth * depth + height * height) / 12}"
-               ixy="0" ixz="0"
-               iyy="${mass * (width * width + height * height) / 12}"
-               iyz="0"
-               izz="${mass * (width * width + depth * depth) / 12}"/>
-    </inertial>
-  </xacro:macro>
-  <!-- Inertia of a thick-walled cylindrical tube with open ends. Height is
-       measured along the z axis, which is the tube's axis. inner_rad and
-       outer_rad are the tube's inner and outer radii, respectively. -->
-  <xacro:macro name="thick_walled_tube_inertial"
-               params="inner_rad outer_rad height mass">
-    <inertial>
-      <mass value="${mass}"/>
-      <inertia ixx="${(1 / 12) * mass * (3 * (inner_rad * inner_rad +
-                    outer_rad * outer_rad) + height * height)}"
-               ixy="0" ixz="0"
-               iyy="${(1 / 12) * mass * (3 * (inner_rad * inner_rad +
-                    outer_rad * outer_rad) + height * height)}"
-               iyz="0"
-               izz="${mass * (inner_rad * inner_rad +
-                    outer_rad * outer_rad) / 2}"/>
-    </inertial>
-  </xacro:macro>
-  <!-- Shock absorber -->
-  <xacro:macro name="shock"
-               params="lr_prefix fr_prefix lr_reflect fr_reflect child">
-    <joint name="${lr_prefix}_${fr_prefix}_shock" type="prismatic">
-      <parent link="chassis"/>
-      <child link="${child}"/>
-      <origin xyz="${fr_reflect * wheelbase / 2}
-                   ${lr_reflect * ((hex_hub_dist / 2) - axle_length)}
-                   ${(wheel_travel / 2) - shock_z_offset}"/>
-      <axis xyz="0 0 -1"/>
-      <limit lower="${-wheel_travel / 2}" upper="${wheel_travel / 2}"
-             effort="${shock_eff_limit}" velocity="${shock_vel_limit}"/>
-    </joint>
-    <transmission name="${lr_prefix}_${fr_prefix}_shock_trans">
-      <type>transmission_interface/SimpleTransmission</type>
-      <joint name="${lr_prefix}_${fr_prefix}_shock">
-        <hardwareInterface>hardware_interface/EffortJointInterface</hardwareInterface>
-      </joint>
-      <actuator name="${lr_prefix}_${fr_prefix}_shock_act">
-        <!-- This hardwareInterface element exists for compatibility
-             with ROS Hydro. -->
-        <hardwareInterface>hardware_interface/EffortJointInterface</hardwareInterface>
-        <mechanicalReduction>1</mechanicalReduction>
-      </actuator>
-    </transmission>
-  </xacro:macro>
-  <!-- The "wheel" macro defines an axle carrier, axle, and wheel. -->
-  <xacro:macro name="wheel" params="lr_prefix fr_prefix lr_reflect tire_dia tire_width hex_hub_depth wheel_mass">
-    <link name="${lr_prefix}_${fr_prefix}_axle_carrier">
-      <xacro:null_inertial/>
-    </link>
-    <!-- The left and right axles have the same axis so that identical
-         rotation values cause the wheels to rotate in the same direction. -->
-    <joint name="${lr_prefix}_${fr_prefix}_axle" type="continuous">
-      <parent link="${lr_prefix}_${fr_prefix}_axle_carrier"/>
-      <child link="${lr_prefix}_${fr_prefix}_wheel"/>
-      <origin rpy="${degrees_90} 0 0"/>
-      <axis xyz="0 0 -1"/>
-      <limit effort="${axle_eff_limit}" velocity="${axle_vel_limit}"/>
-    </joint>
-    <transmission name="${lr_prefix}_${fr_prefix}_axle_trans">
-      <type>transmission_interface/SimpleTransmission</type>
-      <joint name="${lr_prefix}_${fr_prefix}_axle">
-        <hardwareInterface>hardware_interface/EffortJointInterface</hardwareInterface>
-      </joint>
-      <actuator name="${lr_prefix}_${fr_prefix}_axle_act">
-        <!-- This hardwareInterface element exists for compatibility
-             with ROS Hydro. -->
-        <hardwareInterface>hardware_interface/EffortJointInterface</hardwareInterface>
-        <mechanicalReduction>1</mechanicalReduction>
-      </actuator>
-    </transmission>
-    <link name="${lr_prefix}_${fr_prefix}_wheel">
-      <visual>
-        <origin xyz="0
-                     ${lr_reflect * (axle_length - (tire_width /
-                     2 - hex_hub_depth))}
-                     0"/>
-        <geometry>
-          <cylinder radius="${tire_dia / 2}" length="${tire_width}"/>
-        </geometry>
-        <material name="tire_mat"/>
-      </visual>
-      <collision>
-        <origin xyz="0
-                     ${lr_reflect * (axle_length - (tire_width /
-                     2 - hex_hub_depth))}
-                     0"/>
-        <geometry>
-          <cylinder radius="${tire_dia / 2}" length="${tire_width}"/>
-        </geometry>
-      </collision>
-      <xacro:thick_walled_tube_inertial
-          inner_rad="${hub_dia / 2}" outer_rad="${tire_dia / 2}"
-          height="${tire_width}" mass="${wheel_mass}"/>
-    </link>
-    <gazebo reference="${lr_prefix}_${fr_prefix}_wheel">
-      <material>Gazebo/Black</material>
-    </gazebo>
-  </xacro:macro>
-  <!-- Front wheel -->
-  <xacro:macro name="front_wheel"
-               params="lr_prefix fr_prefix lr_reflect fr_reflect">
-    <xacro:shock lr_prefix="${lr_prefix}" fr_prefix="${fr_prefix}"
-                 lr_reflect="${lr_reflect}" fr_reflect="${fr_reflect}"
-                 child="${lr_prefix}_steering_link"/>
-    <link name="${lr_prefix}_steering_link">
-      <xacro:null_inertial/>
-    </link>
-    <joint name="${lr_prefix}_steering_joint" type="revolute">
-      <parent link="${lr_prefix}_steering_link"/>
-      <child link="${lr_prefix}_${fr_prefix}_axle_carrier"/>
-      <axis xyz="0 0 1"/>
-      <limit lower="${-degrees_45}" upper="${degrees_45}"
-             effort="${servo_stall_torque}" velocity="${servo_no_load_speed}"/>
-    </joint>
-    <transmission name="${lr_prefix}_steering_trans">
-      <type>transmission_interface/SimpleTransmission</type>
-      <joint name="${lr_prefix}_steering_joint">
-        <hardwareInterface>hardware_interface/EffortJointInterface</hardwareInterface>
-      </joint>
-      <actuator name="${lr_prefix}_steering_act">
-        <!-- This hardwareInterface element exists for compatibility
-             with ROS Hydro. -->
-        <hardwareInterface>hardware_interface/EffortJointInterface</hardwareInterface>
-        <mechanicalReduction>1</mechanicalReduction>
-      </actuator>
-    </transmission>
-    <xacro:wheel lr_prefix="${lr_prefix}" fr_prefix="${fr_prefix}"
-                 lr_reflect="${lr_reflect}"
-                 tire_dia="${ftire_dia}" tire_width="${ftire_width}"
-                 hex_hub_depth="${fhex_hub_depth}" wheel_mass="${fwheel_mass}"/>
-  </xacro:macro>
-  <!-- Rear wheel -->
-  <xacro:macro name="rear_wheel"
-               params="lr_prefix fr_prefix lr_reflect fr_reflect">
-    <xacro:shock lr_prefix="${lr_prefix}" fr_prefix="${fr_prefix}"
-                 lr_reflect="${lr_reflect}" fr_reflect="${fr_reflect}"
-                 child="${lr_prefix}_${fr_prefix}_axle_carrier"/>
-    <xacro:wheel lr_prefix="${lr_prefix}" fr_prefix="${fr_prefix}"
-                 lr_reflect="${lr_reflect}"
-                 tire_dia="${btire_dia}" tire_width="${btire_width}"
-                 hex_hub_depth="${bhex_hub_depth}" wheel_mass="${bwheel_mass}"/>
-  </xacro:macro>
   <!-- base_link must have geometry so that its axes can be displayed in
        rviz. -->
@@ -246,5 +81,5 @@
   <link name="chassis">
     <visual>
-      <origin xyz="0 0 ${-chassis_height / 2}"/>
+      <origin xyz="${chassis_length / 2} 0 ${chassis_offset}"/> <!--Defualt: 0 0 ${-chassis_height / 2} -->
       <geometry>
         <box size="${chassis_length} ${chassis_width} ${chassis_height}"/>
@@ -253,5 +88,5 @@
     </visual>
     <collision>
-      <origin xyz="0 0 ${-chassis_height / 2}"/>
+      <origin xyz="${chassis_length / 2} 0 ${chassis_offset}"/>
       <geometry>
         <box size="${chassis_length} ${chassis_width} ${chassis_height}"/>
@@ -280,7 +115,6 @@
   <xacro:rear_wheel lr_prefix="right" fr_prefix="rear"
                     lr_reflect="-1" fr_reflect="-1"/>
-  <gazebo>
-    <plugin name="gazebo_ros_control" filename="libgazebo_ros_control.so"/>
-  </gazebo>
+<!-- TODO: Write a macro for sensors -->
+  <!-- Camera -->
   <link name="camera">
     <collision>
@@ -306,13 +140,7 @@
   <joint name="camera_joint" type="fixed">
     <axis xyz="0 1 0" />
-    <origin xyz=".2 0 .3" rpy="0 0 0"/> <!-- CHANGE LATER-->
+    <origin xyz=".2 0 .5" rpy="0 0 0"/> <!-- CHANGE LATER-->
     <parent link="chassis"/>
     <child link="camera"/>
-  </joint>
-  <joint name="hokuyo_joint" type="fixed">
-    <axis xyz="0 1 0" />
-    <origin xyz=".15 0 .2" rpy="0 -.1 0"/> <!-- CHANGE LATER-->
-    <parent link="chassis"/>
-    <child link="hokuyo"/>
   </joint>
   <!-- Hokuyo Laser -->
@@ -336,3 +164,61 @@
     </inertial>
   </link>
+  <joint name="hokuyo_joint" type="fixed">
+    <axis xyz="0 1 0" />
+    <origin xyz=".15 0 .6" rpy="0 -.1 0"/> <!-- CHANGE LATER-->
+    <parent link="chassis"/>
+    <child link="hokuyo"/>
+  </joint>
+  <!-- GPS -->
+  <link name="gps">
+    <collision>
+      <origin xyz="0 0 0" rpy="0 0 0"/>
+      <geometry>
+    <box size="0.1 0.1 0.1"/>
+      </geometry>
+    </collision>
+    <visual>
+      <origin xyz="0 0 0" rpy="0 0 0"/>
+      <geometry>
+        <mesh filename="package://tractor_sim_description/meshes/hokuyo.dae"/><!-- CHANGE LATER-->
+      </geometry>
+    </visual>
+    <inertial>
+      <mass value="1e-5" />
+      <origin xyz="0 0 0" rpy="0 0 0"/>
+      <inertia ixx="1e-6" ixy="0" ixz="0" iyy="1e-6" iyz="0" izz="1e-6" />
+    </inertial>
+  </link>
+  <joint name="gps_joint" type="fixed">
+    <axis xyz="0 1 0" />
+    <origin xyz=".15 0 .7" rpy="0 -.1 0"/> <!-- CHANGE LATER-->
+    <parent link="chassis"/>
+    <child link="gps"/>
+  </joint>
+  <!-- IMU -->
+  <link name="imu">
+    <collision>
+      <origin xyz="0 0 0" rpy="0 0 0"/>
+      <geometry>
+    <box size="0.1 0.1 0.1"/>
+      </geometry>
+    </collision>
+    <visual>
+      <origin xyz="0 0 0" rpy="0 0 0"/>
+      <geometry>
+        <mesh filename="package://tractor_sim_description/meshes/hokuyo.dae"/><!-- CHANGE LATER-->
+      </geometry>
+    </visual>
+    <inertial>
+      <mass value="1e-5" />
+      <origin xyz="0 0 0" rpy="0 0 0"/>
+      <inertia ixx="1e-6" ixy="0" ixz="0" iyy="1e-6" iyz="0" izz="1e-6" />
+    </inertial>
+  </link>
+  <joint name="imu_joint" type="fixed">
+    <axis xyz="0 1 0" />
+    <origin xyz=".15 0 .8" rpy="0 -.1 0"/> <!-- CHANGE LATER-->
+    <parent link="chassis"/>
+    <child link="imu"/>
+  </joint>
 </robot>

Commit message: Added sensor macro

File: tractor_sim_description/urdf/kubo.urdf.xacro (robot description, xacro)
@@ -63,6 +63,6 @@
   <xacro:property name="servo_stall_torque" value="5649"/>
   <xacro:property name="servo_no_load_speed" value="4553"/>
-  <xacro:property name="cameraSize" value="0.05"/>
-  <xacro:property name="cameraMass" value="0.1"/>
+  <xacro:property name="sensorSize" value="0.05"/> <!--TODO: Get rid of this -->
+  <xacro:property name="sensorMass" value="0.1"/>
   <!-- base_link must have geometry so that its axes can be displayed in
        rviz. -->
@@ -115,34 +115,19 @@
   <xacro:rear_wheel lr_prefix="right" fr_prefix="rear"
                     lr_reflect="-1" fr_reflect="-1"/>
-<!-- TODO: Write a macro for sensors -->
   <!-- Camera -->
-  <link name="camera">
-    <collision>
-      <origin xyz="0 0 0" rpy="0 0 0"/>
-      <geometry>
-        <box size="${cameraSize} ${cameraSize} ${cameraSize}"/>
-      </geometry>
-    </collision>
-    <visual>
-      <origin xyz="0 0 0" rpy="0 0 0"/>
-      <geometry>
-        <box size="${cameraSize} ${cameraSize} ${cameraSize}"/>
-      </geometry>
-      <material name="green"/>
-    </visual>
-    <inertial>
-      <mass value="${cameraMass}" />
-      <origin xyz="0 0 0" rpy="0 0 0"/>
-      <box_inertia m="${cameraMass}" x="${cameraSize}" y="${cameraSize}" z="${cameraSize}" />
-      <inertia ixx="1e-6" ixy="0" ixz="0" iyy="1e-6" iyz="0" izz="1e-6" />
-    </inertial>
-  </link>
-  <joint name="camera_joint" type="fixed">
-    <axis xyz="0 1 0" />
-    <origin xyz=".2 0 .5" rpy="0 0 0"/> <!-- CHANGE LATER-->
-    <parent link="chassis"/>
-    <child link="camera"/>
-  </joint>
+  <xacro:sensor sensor_name="camera"
+                x_pos="0" y_pos="0" z_pos="0"
+                x_rot="0" y_rot="0" z_rot="0"/>
+  <xacro:sensor sensor_name="hokuyo"
+                x_pos="0" y_pos="0" z_pos="0"
+                x_rot="0" y_rot="0" z_rot="0"/>
+  <xacro:sensor sensor_name="imu"
+                x_pos="0" y_pos="0" z_pos="0"
+                x_rot="0" y_rot="0" z_rot="0"/>
+  <xacro:sensor sensor_name="gps"
+                x_pos="0" y_pos="0" z_pos="0"
+                x_rot="0" y_rot="0" z_rot="0"/>
   <!-- Hokuyo Laser -->
+  <!-- Using mesh example
   <link name="hokuyo">
     <collision>
@@ -166,59 +151,8 @@
   <joint name="hokuyo_joint" type="fixed">
     <axis xyz="0 1 0" />
-    <origin xyz=".15 0 .6" rpy="0 -.1 0"/> <!-- CHANGE LATER-->
+    <origin xyz=".15 0 .6" rpy="0 -.1 0"/>
     <parent link="chassis"/>
     <child link="hokuyo"/>
   </joint>
-  <!-- GPS -->
-  <link name="gps">
-    <collision>
-      <origin xyz="0 0 0" rpy="0 0 0"/>
-      <geometry>
-    <box size="0.1 0.1 0.1"/>
-      </geometry>
-    </collision>
-    <visual>
-      <origin xyz="0 0 0" rpy="0 0 0"/>
-      <geometry>
-        <mesh filename="package://tractor_sim_description/meshes/hokuyo.dae"/><!-- CHANGE LATER-->
-      </geometry>
-    </visual>
-    <inertial>
-      <mass value="1e-5" />
-      <origin xyz="0 0 0" rpy="0 0 0"/>
-      <inertia ixx="1e-6" ixy="0" ixz="0" iyy="1e-6" iyz="0" izz="1e-6" />
-    </inertial>
-  </link>
-  <joint name="gps_joint" type="fixed">
-    <axis xyz="0 1 0" />
-    <origin xyz=".15 0 .7" rpy="0 -.1 0"/> <!-- CHANGE LATER-->
-    <parent link="chassis"/>
-    <child link="gps"/>
-  </joint>
-  <!-- IMU -->
-  <link name="imu">
-    <collision>
-      <origin xyz="0 0 0" rpy="0 0 0"/>
-      <geometry>
-    <box size="0.1 0.1 0.1"/>
-      </geometry>
-    </collision>
-    <visual>
-      <origin xyz="0 0 0" rpy="0 0 0"/>
-      <geometry>
-        <mesh filename="package://tractor_sim_description/meshes/hokuyo.dae"/><!-- CHANGE LATER-->
-      </geometry>
-    </visual>
-    <inertial>
-      <mass value="1e-5" />
-      <origin xyz="0 0 0" rpy="0 0 0"/>
-      <inertia ixx="1e-6" ixy="0" ixz="0" iyy="1e-6" iyz="0" izz="1e-6" />
-    </inertial>
-  </link>
-  <joint name="imu_joint" type="fixed">
-    <axis xyz="0 1 0" />
-    <origin xyz=".15 0 .8" rpy="0 -.1 0"/> <!-- CHANGE LATER-->
-    <parent link="chassis"/>
-    <child link="imu"/>
-  </joint>
+-->
 </robot>

File: tractor_sim_description/urdf/kubo_macros.urdf.xacro (robot description, xacro)
@@ -193,3 +193,33 @@
                  hex_hub_depth="${bhex_hub_depth}" wheel_mass="${bwheel_mass}"/>
   </macro>
+  <macro name="sensor"
+         params = "sensor_name x_pos y_pos z_pos x_rot y_rot z_rot">
+     <link name="${sensor_name}">
+       <collision>
+         <origin xyz="0 0 0" rpy="0 0 0"/>
+         <geometry>
+           <box size="${sensorSize} ${sensorSize} ${sensorSize}"/> <!-- CHANGE LATER-->
+         </geometry>
+       </collision>
+       <visual>
+         <origin xyz="0 0 0" rpy="0 0 0"/>
+         <geometry>
+           <box size="${sensorSize} ${sensorSize} ${sensorSize}"/>
+         </geometry>
+         <material name="green"/>
+       </visual>
+       <inertial>
+         <mass value="${sensorMass}"/>
+         <origin xyz="0 0 0" rpy="0 0 0"/>
+         <box_inertia m="${sensorMass}" x="${sensorMass}" y="${sensorMass}" z="${sensorMass}" />
+         <inertia ixx="1e-6" ixy="0" ixz="0" iyy="1e-6" iyz="0" izz="1e-6" />
+       </inertial>
+     </link>
+     <joint name="${sensor_name}_joint" type="fixed">
+       <axis xyz="0 1 0" />
+       <origin xyz="${x_pos} ${y_pos} ${z_pos}" rpy="${x_rot} ${y_rot} ${z_rot}"/> <!-- CHANGE LATER-->
+       <parent link="base_link"/>
+       <child link="${sensor_name}"/>
+     </joint>
+  </macro>
 </robot>

Commit message: made more robust

File: tractor_sim_description/urdf/kubo.urdf.xacro (robot description, xacro)
@@ -11,5 +11,5 @@
       Note: Size of chassis won't affect wheel position or function-->
   <xacro:property name="chassis_length" value="1.5"/>
-  <xacro:property name="chassis_width" value="0.6"/>
+  <xacro:property name="chassis_width" value="0.3"/>
   <xacro:property name="chassis_height" value="0.1"/>
   <xacro:property name="chassis_mass" value="2.788"/>
@@ -20,5 +20,5 @@
        is a "zero offset" wheel. hex_hub_depth = tire_width / 2 -
        axle_length. -->
-  <xacro:property name="hub_dia" value="0.09652"/> <!-- ? -->
+  <xacro:property name="hub_dia" value="0.09652"/> <!-- For inertia measurements -->
   <xacro:property name="ftire_dia" value="0.5"/>
   <xacro:property name="ftire_width" value="0.15"/>

Commit message: Made diagrams, moving to another branch to try simplifying links. Everything here works but there are a lot of unneccessary components (i.e. shocks, hubs, etc.)

File: tractor_sim_description/urdf/kubo.urdf.xacro (robot description, xacro)
@@ -34,6 +34,6 @@
        vertical wheel travel. -->
   <xacro:property name="wheelbase" value="1.5"/>
-  <xacro:property name="hex_hub_dist" value="1.4"/> <!-- ? -->
-  <xacro:property name="axle_length" value="0.3"/> <!-- ? -->
+  <xacro:property name="hex_hub_dist" value="1.4"/> <!-- ? Default: 1.4-->
+  <xacro:property name="axle_length" value="0.3"/> <!-- ? Default: 0.3 -->
   <xacro:property name="wheel_travel" value="0"/>
   <xacro:property name="shock_z_offset" value="0.0655"/>
