Commit message: Added comments, removed unneccessary parameters

File: tractor_sim_description/urdf/kubo.urdf.xacro (robot description, xacro)
@@ -7,43 +7,51 @@
   <xacro:property name="degrees_45" value="0.785398163"/>
   <xacro:property name="degrees_90" value="1.57079633"/>
+  <!-- For documentation for visual of what these parameters are, see repo -->
   <!-- chassis_length is measured along the x axis, chassis_width
        along the y axis, and chassis_height along the z axis.
-      Note: Size of chassis won't affect wheel position or function-->
+       Note: Size of chassis won't affect wheel position or function, so be
+       careful about making it too big-->
+  <!--Length of chassis (m) -->
   <xacro:property name="chassis_length" value="1.5"/>
+  <!--Width of chassis (m) -->
   <xacro:property name="chassis_width" value="0.3"/>
+  <!--Height of chassis (m) -->
   <xacro:property name="chassis_height" value="0.1"/>
+  <!--Mass of chassis (kg) -->
   <xacro:property name="chassis_mass" value="2.788"/>
-  <xacro:property name="chassis_offset" value=".25"/> <!-- Z Distance from ground -->
-  <!-- hub_dia and tire_dia are the diameters of the hub and tire,
-       respectively. hex_hub_depth is the distance that the hex hub is
-       inset from the outer edge of the tire. It is set so that each wheel
-       is a "zero offset" wheel. hex_hub_depth = tire_width / 2 -
-       axle_length. -->
-  <xacro:property name="hub_dia" value="0.09652"/> <!-- For inertia measurements -->
+  <!-- Z Distance from ground (m) -->
+  <xacro:property name="chassis_offset" value=".25"/>
+  <!-- Distance from center of front tire to center of back tire measured parallel to floor (m) -->
+  <xacro:property name="wheelbase" value="1.5"/>
+  <!-- Front tire diameter (m) -->
   <xacro:property name="ftire_dia" value="0.5"/>
+  <!-- Front tire width (m) -->
   <xacro:property name="ftire_width" value="0.15"/>
-  <xacro:property name="fhex_hub_depth" value="${ftire_width / 2 - axle_length}"/> <!-- tire_width / 2 - axle_length-->
+  <!-- Front tire mass (kg) -->
   <xacro:property name="fwheel_mass" value="0.29"/>
+  <!-- Distance between front wheels (inner side of wheel)-->
+  <xacro:property name="fwheel_dist" value="0.8"/>
+  <!-- Back tire diameter (m) -->
   <xacro:property name="btire_dia" value="0.7"/>
+  <!-- Back tire width (m) -->
   <xacro:property name="btire_width" value="0.2"/>
-  <xacro:property name="bhex_hub_depth" value="${btire_width / 2 - axle_length}"/> <!-- tire_width / 2 - axle_length-->
+  <!-- Back tire mass (kg) -->
   <xacro:property name="bwheel_mass" value="0.29"/>
-  <!-- hex_hub_dist is the distance between left and right hex hubs when
-       the shock absorbers are fully extended. axle_length is the distance
-       from a U joint to the corresponding hex hub. wheel_travel is the
-       vertical wheel travel. -->
-  <xacro:property name="wheelbase" value="1.5"/>
-  <xacro:property name="hex_hub_dist" value="1.4"/> <!-- ? Default: 1.4-->
-  <xacro:property name="axle_length" value="0.3"/> <!-- ? Default: 0.3 -->
+  <!-- Distance between back wheels (inner side of wheel)-->
+  <xacro:property name="bwheel_dist" value="0.8"/>
+  <!-- Other parameters - currently not used to improve simulation -->
+  <!-- Inner diameter of tire, used for inertia measurements. 0 indicates a solid cylinder -->
+  <xacro:property name="hub_dia" value="0.0"/>
+  <!-- For vehicles with suspension, this is how much the wheels can move up and down -->
   <xacro:property name="wheel_travel" value="0"/>
+  <!-- For vehicles with suspension, this sets where the suspension is mounted -->
   <xacro:property name="shock_z_offset" value="0.0655"/>
   <!-- shock_eff_limit is 2 * ((shock_stroke / 2) * shock_spring_constant) N.
-       shock_stroke is 0.028575 meters. shock_spring_constant, an approximation
-       of a Traxxas Ultra Shock shock absorber spring's constant, is
-       437.817 N/m. -->
-  <xacro:property name="shock_eff_limit" value="125106"/>
+       shock_stroke is 0.028575 meters. shock_spring_constant is the shock
+       absorber spring's constant in units of N/m. Currently set to arbitrary
+       high values to disable shocks behavior  -->
+  <xacro:property name="shock_eff_limit" value="1000000"/>
   <xacro:property name="shock_vel_limit" value="1000000"/>
-  <!-- The specifications for a Titan(R) 550 motor could not be found, so the
-       stall torque of a Mabuchi Motor(R) RS-550VC-7525 motor was used instead.
+  <!-- Sample calculations for stall torque of a Mabuchi Motor(R) RS-550VC-7525 motor
        num_spur_gear_teeth = 68
        num_pinion_gear_teeth = 19
@@ -58,9 +66,8 @@
   <xacro:property name="axle_eff_limit" value="512766"/>
   <xacro:property name="axle_vel_limit" value="2448696"/>
-  <!-- These constants are used to simulate a Traxxas 2056 servo operated at
-       6 V. servo_stall_torque is measured in N m. servo_no_load_speed is
+  <!-- motor_stall_torque is measured in N m. motor_no_load_speed is
        measured in rad/s. -->
-  <xacro:property name="servo_stall_torque" value="5649"/>
-  <xacro:property name="servo_no_load_speed" value="4553"/>
+  <xacro:property name="motor_stall_torque" value="5649"/>
+  <xacro:property name="motor_no_load_speed" value="4553"/>
   <xacro:property name="sensorSize" value="0.05"/> <!--TODO: Get rid of this -->
   <xacro:property name="sensorMass" value="0.1"/>
@@ -81,5 +88,5 @@
   <link name="chassis">
     <visual>
-      <origin xyz="${chassis_length / 2} 0 ${chassis_offset}"/> <!--Defualt: 0 0 ${-chassis_height / 2} -->
+      <origin xyz="${chassis_length / 2} 0 ${chassis_offset}"/>
       <geometry>
         <box size="${chassis_length} ${chassis_width} ${chassis_height}"/>
@@ -116,5 +123,6 @@
                     lr_reflect="-1" fr_reflect="-1"/>
   <!-- Sensors -->
-  <!-- IMU approximate
+  <!-- Sensor positions are relative to base_link
+  IMU approximate
 https://github.com/olinrobotics/gravl/wiki/Kubo:-Transforms-->
   <xacro:sensor sensor_name="camera"

File: tractor_sim_description/urdf/kubo_macros.urdf.xacro (robot description, xacro)
@@ -47,5 +47,5 @@
       <child link="${child}"/>
       <origin xyz="${fr_reflect * wheelbase / 2 + (wheelbase/2)}
-                   ${lr_reflect * ((hex_hub_dist / 2) - axle_length)}
+                   ${lr_reflect * (bwheel_dist / 2)}
                    ${(btire_dia / 2)}"/> <!-- Default: ${fr_reflect * wheelbase / 2}
                                 ${lr_reflect * ((hex_hub_dist / 2) - axle_length)}
@@ -74,5 +74,5 @@
       <child link="${child}"/>
       <origin xyz="${fr_reflect * wheelbase / 2 + (wheelbase/2)}
-                   ${lr_reflect * ((hex_hub_dist / 2) - axle_length)}
+                   ${lr_reflect * (fwheel_dist / 2)}
                    ${(ftire_dia / 2)}"/> <!-- Default: ${fr_reflect * wheelbase / 2}
                                 ${lr_reflect * ((hex_hub_dist / 2) - axle_length)}
@@ -96,5 +96,5 @@
   </xacro:macro>
   <!-- The "wheel" macro defines an axle carrier, axle, and wheel. -->
-  <xacro:macro name="wheel" params="lr_prefix fr_prefix lr_reflect tire_dia tire_width hex_hub_depth wheel_mass">
+  <xacro:macro name="wheel" params="lr_prefix fr_prefix lr_reflect tire_dia tire_width wheel_mass">
     <link name="${lr_prefix}_${fr_prefix}_axle_carrier">
       <null_inertial/>
@@ -124,6 +124,6 @@
       <visual>
         <origin xyz="0
-                     ${lr_reflect * (axle_length - (tire_width /
-                     2 - hex_hub_depth))}
+                     ${lr_reflect * (- (tire_width /
+                     2 - (tire_width / 2)))}
                      0"/>
         <geometry>
@@ -134,6 +134,6 @@
       <collision>
         <origin xyz="0
-                     ${lr_reflect * (axle_length - (tire_width /
-                     2 - hex_hub_depth))}
+                     ${lr_reflect * (- (tire_width /
+                     2 - (tire_width / 2)))}
                      0"/>
         <geometry>
@@ -163,5 +163,5 @@
       <axis xyz="0 0 1"/>
       <limit lower="${-degrees_45}" upper="${degrees_45}"
-             effort="${servo_stall_torque}" velocity="${servo_no_load_speed}"/>
+             effort="${motor_stall_torque}" velocity="${motor_no_load_speed}"/>
     </joint>
     <transmission name="${lr_prefix}_steering_trans">
@@ -180,5 +180,5 @@
                  lr_reflect="${lr_reflect}"
                  tire_dia="${ftire_dia}" tire_width="${ftire_width}"
-                 hex_hub_depth="${fhex_hub_depth}" wheel_mass="${fwheel_mass}"/>
+                 wheel_mass="${fwheel_mass}"/>
   </xacro:macro>
   <!-- Rear wheel -->
@@ -191,5 +191,5 @@
                  lr_reflect="${lr_reflect}"
                  tire_dia="${btire_dia}" tire_width="${btire_width}"
-                 hex_hub_depth="${bhex_hub_depth}" wheel_mass="${bwheel_mass}"/>
+                 wheel_mass="${bwheel_mass}"/>
   </xacro:macro>
   <xacro:macro name="sensor"

Commit message: Added mesh to tractor

File: tractor_sim_description/urdf/kubo.urdf.xacro (robot description, xacro)
@@ -1,6 +1,8 @@
 <?xml version="1.0"?>
+<!-- TODO: double check parameters. If correct, then shape meshes to look better -->
+<!-- TODO: add meshes for sensors -->
+<!-- TODO: add box blade -->
 <robot name="kubo" xmlns:xacro="http://www.ros.org/wiki/xacro">
   <xacro:include filename="$(find tractor_sim_description)/urdf/kubo.gazebo"/>
-  <xacro:include filename="$(find tractor_sim_description)/urdf/kubo_materials.urdf.xacro"/>
   <xacro:include filename="$(find tractor_sim_description)/urdf/kubo_macros.urdf.xacro"/>
   <!-- Degree-to-radian conversions -->
@@ -13,5 +15,5 @@
        careful about making it too big-->
   <!--Length of chassis (m) -->
-  <xacro:property name="chassis_length" value="1.5"/>
+  <xacro:property name="chassis_length" value="1.1"/>
   <!--Width of chassis (m) -->
   <xacro:property name="chassis_width" value="0.3"/>
@@ -23,5 +25,5 @@
   <xacro:property name="chassis_offset" value=".25"/>
   <!-- Distance from center of front tire to center of back tire measured parallel to floor (m) -->
-  <xacro:property name="wheelbase" value="1.5"/>
+  <xacro:property name="wheelbase" value="1.2"/>
   <!-- Front tire diameter (m) -->
   <xacro:property name="ftire_dia" value="0.5"/>
@@ -79,5 +81,4 @@
         <box size="0.01 0.01 0.01"/>
       </geometry>
-      <material name="chassis_mat"/>
     </visual>
   </link>
@@ -88,4 +89,11 @@
   <link name="chassis">
     <visual>
+      <origin xyz="${chassis_length/2} 0 0" rpy="0 0 ${2*degrees_90}" scale="1 1 1"/>
+      <geometry>
+        <mesh filename="package://tractor_sim_description/meshes/kubo_chassis.dae"/>
+      </geometry>
+    </visual>
+    <!--
+    <visual>
       <origin xyz="${chassis_length / 2} 0 ${chassis_offset}"/>
       <geometry>
@@ -94,4 +102,5 @@
       <material name="chassis_mat"/>
     </visual>
+  -->
     <collision>
       <origin xyz="${chassis_length / 2} 0 ${chassis_offset}"/>
@@ -106,7 +115,4 @@
     </xacro:solid_cuboid_inertial>
   </link>
-  <gazebo reference="chassis">
-    <material>Gazebo/Grey</material>
-  </gazebo>
   <joint name="base_link_to_chassis" type="fixed">
     <parent link="base_link"/>

File: tractor_sim_description/urdf/kubo_macros.urdf.xacro (robot description, xacro)
@@ -96,5 +96,5 @@
   </xacro:macro>
   <!-- The "wheel" macro defines an axle carrier, axle, and wheel. -->
-  <xacro:macro name="wheel" params="lr_prefix fr_prefix lr_reflect tire_dia tire_width wheel_mass">
+  <xacro:macro name="wheel" params="lr_prefix fr_prefix lr_reflect tire_dia tire_width wheel_mass mesh_file">
     <link name="${lr_prefix}_${fr_prefix}_axle_carrier">
       <null_inertial/>
@@ -126,9 +126,9 @@
                      ${lr_reflect * (- (tire_width /
                      2 - (tire_width / 2)))}
-                     0"/>
-        <geometry>
-          <cylinder radius="${tire_dia / 2}" length="${tire_width}"/>
-        </geometry>
-        <material name="tire_mat"/>
+                     0"
+                rpy="${lr_reflect * degrees_90} 0 0"/>
+       <geometry>
+         <mesh filename="${mesh_file}"/>
+       </geometry>
       </visual>
       <collision>
@@ -145,7 +145,4 @@
           height="${tire_width}" mass="${wheel_mass}"/>
     </link>
-    <gazebo reference="${lr_prefix}_${fr_prefix}_wheel">
-      <material>Gazebo/Black</material>
-    </gazebo>
   </xacro:macro>
   <!-- Front wheel -->
@@ -180,5 +177,6 @@
                  lr_reflect="${lr_reflect}"
                  tire_dia="${ftire_dia}" tire_width="${ftire_width}"
-                 wheel_mass="${fwheel_mass}"/>
+                 wheel_mass="${fwheel_mass}"
+                 mesh_file = "package://tractor_sim_description/meshes/kubo_front_tire.dae"/>
   </xacro:macro>
   <!-- Rear wheel -->
@@ -191,5 +189,6 @@
                  lr_reflect="${lr_reflect}"
                  tire_dia="${btire_dia}" tire_width="${btire_width}"
-                 wheel_mass="${bwheel_mass}"/>
+                 wheel_mass="${bwheel_mass}"
+                 mesh_file = "package://tractor_sim_description/meshes/kubo_back_tire.dae"/>
   </xacro:macro>
   <xacro:macro name="sensor"
@@ -207,5 +206,4 @@
            <box size="${sensorSize} ${sensorSize} ${sensorSize}"/>
          </geometry>
-         <material name="green"/>
        </visual>
        <inertial>

Commit message: derp backflip code

File: tractor_sim_description/urdf/kubo.urdf.xacro (robot description, xacro)
@@ -119,4 +119,27 @@
     <child link="chassis"/>
   </joint>
+  <!-- Hitch -->
+  <link name="hitch">
+    <visual>
+      <origin xyz="0 0 0" rpy="0 ${degrees_90} ${2*degrees_90}" scale="1 1 1"/>
+      <geometry>
+        <box size="${chassis_length} ${chassis_width} ${chassis_height}"/>
+      </geometry>
+      <!-- <geometry>
+        <mesh filename="package://tractor_sim_description/meshes/kubo_chassis.dae"/>
+      </geometry> -->
+    </visual>
+    <xacro:solid_cuboid_inertial
+        width="${chassis_length}" depth="${chassis_width}"
+        height="${chassis_height}" mass="${chassis_mass}">
+      <origin xyz="0 0 ${-chassis_height / 2}"/>
+    </xacro:solid_cuboid_inertial>
+  </link>
+  <joint name="base_link_to_hitch" type="prismatic">
+    <parent link="base_link"/>
+    <child link="hitch"/>
+    <limit effort="1000.0" lower="-0.38" upper="0" velocity="0.5"/>
+    <origin xyz="0 0 0" rpy="0 ${degrees_90} 0"/>
+  </joint>
   <!-- Wheels -->
   <xacro:front_wheel lr_prefix="left" fr_prefix="front"

Commit message: current progress

File: tractor_sim_description/urdf/kubo.urdf.xacro (robot description, xacro)
@@ -140,5 +140,5 @@
     <child link="hitch"/>
     <limit effort="1000.0" lower="-0.38" upper="0" velocity="0.5"/>
-    <origin xyz="0 0 0" rpy="0 ${degrees_90} 0"/>
+    <origin xyz="0 0 0" rpy="0 0 0"/>
   </joint>
   <!-- Wheels -->

Commit message: Create box blade, add mesh, add height setting behavior

File: tractor_sim_description/urdf/kubo.urdf.xacro (robot description, xacro)
@@ -122,15 +122,15 @@
   <link name="hitch">
     <visual>
-      <origin xyz="0 0 0" rpy="0 ${degrees_90} ${2*degrees_90}" scale="1 1 1"/>
-      <geometry>
+      <origin xyz="0 0 0" rpy="${degrees_90} 0 ${-degrees_90}" scale="1 1 1"/>
+      <!-- <geometry>
         <box size="${chassis_length} ${chassis_width} ${chassis_height}"/>
-      </geometry>
-      <!-- <geometry>
-        <mesh filename="package://tractor_sim_description/meshes/kubo_chassis.dae"/>
       </geometry> -->
+      <geometry>
+        <mesh filename="package://tractor_sim_description/meshes/blade.dae"/>
+      </geometry>
     </visual>
     <xacro:solid_cuboid_inertial
         width="${chassis_length}" depth="${chassis_width}"
-        height="${chassis_height}" mass="${chassis_mass}">
+        height="${chassis_height}" mass="0.1">
       <origin xyz="0 0 ${-chassis_height / 2}"/>
     </xacro:solid_cuboid_inertial>
@@ -139,6 +139,6 @@
     <parent link="base_link"/>
     <child link="hitch"/>
-    <limit effort="1000.0" lower="-0.38" upper="0" velocity="0.5"/>
-    <origin xyz="0 0 0" rpy="0 0 0"/>
+    <limit effort="10" lower="-0.25" upper="0.1" velocity="0.1"/>
+    <origin xyz="-0.5 0 0.1" rpy="0 ${degrees_90} 0"/>
   </joint>
   <!-- Wheels -->

Commit message: Add limits to hitch

File: tractor_sim_description/urdf/kubo.urdf.xacro (robot description, xacro)
@@ -139,6 +139,6 @@
     <parent link="base_link"/>
     <child link="hitch"/>
-    <limit effort="10" lower="-0.25" upper="0.1" velocity="0.1"/>
-    <origin xyz="-0.5 0 0.1" rpy="0 ${degrees_90} 0"/>
+    <limit effort="10" lower="-1" upper="1" velocity="0.1"/>
+    <origin xyz="-0.5 0 -0.3" rpy="0 ${degrees_90} 0"/>
   </joint>
   <!-- Wheels -->

Commit message: create 3d lidar in simulation, need to match it to the specs of lidarx and tractor

File: tractor_sim_description/urdf/kubo.urdf.xacro (robot description, xacro)
@@ -6,4 +6,5 @@
   <xacro:include filename="$(find tractor_sim_description)/urdf/kubo.gazebo"/>
   <xacro:include filename="$(find tractor_sim_description)/urdf/kubo_macros.urdf.xacro"/>
+  <xacro:include filename="$(find tractor_sim_description)/urdf/lidarx.urdf.xacro"/>
   <!-- Degree-to-radian conversions -->
   <xacro:property name="degrees_45" value="0.785398163"/>
@@ -156,24 +157,27 @@
 https://github.com/olinrobotics/gravl/wiki/Kubo:-Transforms-->
   <!-- Make sure names match gravl localization.launch -->
-  <xacro:sensor sensor_name="camera"
+  <xacro:gravl_sensor sensor_name="camera"
                 x_pos="2.08" y_pos="0" z_pos="1.04"
                 x_rot="0" y_rot="0" z_rot="0"/>
-  <xacro:sensor sensor_name="hokuyo-ust-10lx"
+  <!--
+  <xacro:gravl_sensor sensor_name="hokuyo-ust-10lx"
                 x_pos="2.02" y_pos="0" z_pos="1.19"
-                x_rot="0" y_rot="1.5" z_rot="0"/> <!-- testing downward LiDar -->
-                <!-- x_rot="0" y_rot="0.157" z_rot="0" -->
-  <xacro:sensor sensor_name="hokuyo-uxm-30lx-e"
+                x_rot="0" y_rot="1.5" z_rot="0"/>
+  <xacro:gravl_sensor sensor_name="hokuyo-uxm-30lx-e"
                 x_pos="2.02" y_pos="0" z_pos="1.25"
-                x_rot="0" y_rot="0" z_rot="0"/> <!-- testing downward LiDar -->
-                <!-- x_rot="0" y_rot="0.157" z_rot="0" -->
-  <xacro:sensor sensor_name="imu"
+                x_rot="0" y_rot="0" z_rot="0"/>
+  -->
+  <xacro:gravl_sensor sensor_name="imu"
                 x_pos="-0.3" y_pos="0" z_pos="1"
                 x_rot="0" y_rot="0" z_rot="0"/>
-  <xacro:sensor sensor_name="hemisphere_gps"
+  <xacro:gravl_sensor sensor_name="hemisphere_gps"
                 x_pos="1.94" y_pos="0" z_pos="1.49"
                 x_rot="0" y_rot="0" z_rot="0"/>
-  <xacro:sensor sensor_name="gps"
+  <xacro:gravl_sensor sensor_name="gps"
                 x_pos="0.3" y_pos="0" z_pos="2.21"
                 x_rot="0" y_rot="0" z_rot="0"/>
+  <xacro:lidarx name="3d_lidar" gpu="true"
+                x_pos="2.5" y_pos="0" z_pos="1.25"
+                x_rot="0" y_rot="1.5" z_rot="0"/>
   <!-- Hokuyo Laser -->
   <!-- Using mesh example

File: tractor_sim_description/urdf/kubo_macros.urdf.xacro (robot description, xacro)
@@ -192,5 +192,5 @@
                  mesh_file = "package://tractor_sim_description/meshes/kubo_back_tire.dae"/>
   </xacro:macro>
-  <xacro:macro name="sensor"
+  <xacro:macro name="gravl_sensor"
          params = "sensor_name x_pos y_pos z_pos x_rot y_rot z_rot">
      <link name="${sensor_name}">
