Commit message: Change 3D lidar type from gpu to regular, add velodyne simulator as dependency to readme

File: tractor_sim_description/urdf/kubo.urdf.xacro (robot description, xacro)
@@ -160,12 +160,4 @@
                 x_pos="2.08" y_pos="0" z_pos="1.04"
                 x_rot="0" y_rot="0" z_rot="0"/>
-  <!--
-  <xacro:gravl_sensor sensor_name="hokuyo-ust-10lx"
-                x_pos="2.02" y_pos="0" z_pos="1.19"
-                x_rot="0" y_rot="1.5" z_rot="0"/>
-  <xacro:gravl_sensor sensor_name="hokuyo-uxm-30lx-e"
-                x_pos="2.02" y_pos="0" z_pos="1.25"
-                x_rot="0" y_rot="0" z_rot="0"/>
-  -->
   <xacro:gravl_sensor sensor_name="imu"
                 x_pos="-0.3" y_pos="0" z_pos="1"
@@ -177,7 +169,7 @@
                 x_pos="0.3" y_pos="0" z_pos="2.21"
                 x_rot="0" y_rot="0" z_rot="0"/>
-  <xacro:lidarx name="3d_lidar" gpu="true"
-                x_pos="2.5" y_pos="0" z_pos="1.25"
-                x_rot="0" y_rot="1.5" z_rot="0"/>
+  <xacro:lidarx parent="base_link" name="lidarx" topic="/lidarx_points" hz="10" samples="440">
+    <origin xyz="2.5 0 1.25" rpy="0 0.5 0" />
+  </xacro:lidarx>
   <!-- Hokuyo Laser -->
   <!-- Using mesh example

File: tractor_sim_description/urdf/lidarx.urdf.xacro (robot description, xacro)
@@ -1,16 +1,16 @@
 <?xml version="1.0"?>
-<robot xmlns:xacro="http://www.ros.org/wiki/xacro" name="lidarx">
+<robot xmlns:xacro="http://www.ros.org/wiki/xacro" name="VLP-16">
   <xacro:property name="M_PI" value="3.1415926535897931" />
-  <xacro:macro name="lidarx"
-        params="parent:=base_link name:=lidarx topic:=/lidarx_points hz:=10 lasers:=31 samples:=1875 collision_range:=0.3 min_range:=0.9 max_range:=130.0 noise:=0.008 min_angle:=-${M_PI} max_angle:=${M_PI} gpu:=true x_pos:=0 y_pos:=0 z_pos:=0 x_rot:=0 y_rot:=0 z_rot:=0">
-  <joint name="${name}_base_mount_joint" type="fixed">
-    <parent link="${parent}"/>
-    <origin xyz="${x_pos} ${y_pos} ${z_pos}" rpy="${x_rot} ${y_rot} ${z_rot}" />
-    <child link="${name}_base_link"/>
-  </joint>
+  <xacro:macro name="lidarx" params="*origin parent:=base_link name:=lidarx topic:=/lidarx_points hz:=10 lasers:=16 samples:=1875 collision_range:=0.3 min_range:=0.9 max_range:=130.0 noise:=0.008 min_angle:=-${M_PI} max_angle:=${M_PI}">
+    <!-- TODO: Update specs -->
+    <joint name="${name}_base_mount_joint" type="fixed">
+      <xacro:insert_block name="origin" />
+      <parent link="${parent}"/>
+      <child link="${name}_base_link"/>
+    </joint>
     <link name="${name}_base_link">
       <inertial>
         <mass value="0.83"/>
-        <origin xyz="0 0 0" rpy="0 0 0"/>
+        <origin xyz="0 0 0.03585"/>
         <inertia ixx="${(0.83 * (3.0*0.0516*0.0516 + 0.0717*0.0717)) / 12.0}" ixy="0" ixz="0"
           iyy="${(0.83 * (3.0*0.0516*0.0516 + 0.0717*0.0717)) / 12.0}" iyz="0"
@@ -28,5 +28,5 @@
       </visual>
       <collision>
-        <origin rpy="0 0 0" xyz="0 0 0"/>
+        <origin rpy="0 0 0" xyz="0 0 0.03585"/>
         <geometry>
           <cylinder radius="0.0516" length="0.0717"/>
@@ -35,5 +35,6 @@
     </link>
     <joint name="${name}_base_scan_joint" type="fixed" >
-        <parent link="${name}_base_link" />
+      <origin xyz="0 0 0.0377" rpy="0 0 0" />
+      <parent link="${name}_base_link" />
       <child link="${name}"/>
     </joint>
@@ -51,6 +52,7 @@
       </visual>
     </link>
+    <!-- Gazebo requires the velodyne_gazebo_plugins package -->
     <gazebo reference="${name}">
-        <sensor type="gpu_ray" name="${name}-lidarx">
+        <sensor type="ray" name="${name}-lidarx">
           <pose>0 0 0 0 0 0</pose>
           <visualize>false</visualize>
@@ -67,6 +69,6 @@
                 <samples>${lasers}</samples>
                 <resolution>1</resolution>
-                <min_angle>-${15.0*M_PI/180.0}</min_angle>
-                <max_angle> ${15.0*M_PI/180.0}</max_angle>
+                <min_angle>-${20.0*M_PI/180.0}</min_angle>
+                <max_angle> ${20.0*M_PI/180.0}</max_angle>
               </vertical>
             </scan>
@@ -82,5 +84,5 @@
             </noise>
           </ray>
-          <plugin name="gazebo_ros_laser_controller" filename="libgazebo_ros_velodyne_gpu_laser.so">
+          <plugin name="gazebo_ros_laser_controller" filename="libgazebo_ros_velodyne_laser.so">
             <topicName>${topic}</topicName>
             <frameName>${name}</frameName>
